File: etb-9201.kicad_sch (KiCad schematic)
At the start: 5 parts, among them U3 TLE9201SG

Commit message: BOM cleanup, minor USB improvements, bump to 1.2
Parts:
- C3, C4, C5, R5: LCSC_ext 0 -> (none)
- U3: LCSC_ext 1 -> (none); possible_not_ext 1 -> (none)
Other:
- company: FutureProofPerformance.com -> github.com/FOME-Tech
- title: Polygonus Universal 88p -> FOME Universal 112 pin ECU base
Changed lines of the file:
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@@
 	(paper "A4")
 	(title_block
-		(title "Polygonus Universal 88p")
-		(date "2023-11-12")
-		(rev "v1.0")
-		(company "FutureProofPerformance.com")
+		(title "FOME Universal 112 pin ECU base")
+		(date "2026-03-03")
+		(rev "v1.2")
+		(company "github.com/FOME-Tech")
+		(comment 1 "FutureProofPerformance.com")
+		(comment 2 "happycactusgarage.com")
 	)
 	(text "IFX9201 also acceptable"
@@
 			)
 		)
-		(property "LCSC_ext" "0"
-			(at 68.58 57.15 0)
-			(effects
-				(font
-					(size 1.27 1.27)
-				)
-				(hide yes)
-			)
-		)
 		(pin "1"
 		)
@@
 			)
 		)
-		(property "LCSC_ext" "1"
-			(at 97.79 63.5 0)
-			(effects
-				(font
-					(size 1.27 1.27)
-				)
-				(hide yes)
-			)
-		)
-		(property "possible_not_ext" "1"
-			(at 97.79 63.5 0)
-			(effects
-				(font
-					(size 1.27 1.27)
-				)
-				(hide yes)
-			)
-		)
 		(pin "1"
 		)
@@
 			)
 		)
-		(property "LCSC_ext" "0"
-			(at 114.3 60.325 0)
-			(effects
-				(font
-					(size 1.27 1.27)
-				)
-				(hide yes)
-			)
-		)
 		(pin "1"
 		)
@@
 		)
 		(property "LCSC" "C13585"
-			(at 80.645 46.99 0)
-			(effects
-				(font
-					(size 1.27 1.27)
-				)
-				(hide yes)
-			)
-		)
-		(property "LCSC_ext" "0"
 			(at 80.645 46.99 0)
 			(effects
@@
 			(at 114.3 48.895 0)
 			(effects
-				(font
-					(size 1.27 1.27)
-				)
-				(hide yes)
-			)
-		)
-		(property "LCSC_ext" "0"
-			(at 114.3 48.895 0)
-			(effects
