File: wbo-can-trans.kicad_sch (KiCad schematic)
At the start: 7 parts, among them U20 TJA1051T-3

Commit message: BOM cleanup, minor USB improvements, bump to 1.2
Other:
- company: FutureProofPerformance.com -> github.com/FOME-Tech
- title: Polygonus Universal 88p -> FOME Universal 112 pin ECU base
Changed lines of the file:
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@@
 	(paper "A4")
 	(title_block
-		(title "Polygonus Universal 88p")
-		(date "2023-11-12")
-		(rev "v1.0")
-		(company "FutureProofPerformance.com")
+		(title "FOME Universal 112 pin ECU base")
+		(date "2026-03-03")
+		(rev "v1.2")
+		(company "github.com/FOME-Tech")
+		(comment 1 "FutureProofPerformance.com")
+		(comment 2 "happycactusgarage.com")
 	)
 	(text "n.p."
