File: vr_module_poly.kicad_sch (KiCad schematic)
At the start: 43 parts, among them U4 SRV05-4, U5 74HC02, U6 MCP6004, U7 MAX9142, U8 NC7SB3157P6X, U9 NC7SB3157P6X

Commit message: BOM cleanup, minor USB improvements, bump to 1.2
Other:
- company: (none) -> github.com/FOME-Tech
- title: (none) -> FOME Universal 112 pin ECU base
Changed lines of the file:
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@@
 	(generator_version "9.0")
 	(paper "A4")
+	(title_block
+		(title "FOME Universal 112 pin ECU base")
+		(date "2026-03-03")
+		(rev "v1.2")
+		(company "github.com/FOME-Tech")
+		(comment 1 "FutureProofPerformance.com")
+		(comment 2 "happycactusgarage.com")
+	)
 	(text "RS Latch\nTracks which edge happened last"
 		(exclude_from_sim no)

Commit message: more BOM optimization
Parts:
- U8, U9: LCSC C87403 -> C36533657
Changed lines of the file:
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@@
 			)
 		)
-		(property "LCSC" "C87403"
+		(property "LCSC" "C36533657"
 			(at 163.83 35.56 0)
 			(effects
@@
 			)
 		)
-		(property "LCSC" "C87403"
+		(property "LCSC" "C36533657"
 			(at 199.39 33.02 0)
 			(effects
@@
 			)
 		)
-		(property "LCSC" "C87403"
+		(property "LCSC" "C36533657"
 			(at 163.83 105.41 0)
 			(effects
@@
 			)
 		)
-		(property "LCSC" "C87403"
+		(property "LCSC" "C36533657"
 			(at 213.36 33.02 0)
 			(effects
