File: Lowside Adder.kicad_sch (KiCad schematic)
At the start: 10 parts, among them U11 VNL5090, U12 VNL5090, U13 VNL5090, U14 VNL5090

Commit message: BOM cleanup, minor USB improvements, bump to 1.2
Parts:
- D2, D3, D4, D5: LCSC (none) -> C8678
- RN1, RN2: LCSC_ext 0 -> (none)
Other:
- company: FutureProofPerformance.com -> github.com/FOME-Tech
- title: Polygonus Universal 88p -> FOME Universal 112 pin ECU base
Changed lines of the file:
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@@
 	(paper "A4")
 	(title_block
-		(title "Polygonus Universal 88p")
-		(date "2023-11-12")
-		(rev "v1.0")
-		(company "FutureProofPerformance.com")
+		(title "FOME Universal 112 pin ECU base")
+		(date "2026-03-03")
+		(rev "v1.2")
+		(company "github.com/FOME-Tech")
+		(comment 1 "FutureProofPerformance.com")
+		(comment 2 "happycactusgarage.com")
 	)
 	(junction
@@
 			)
 		)
+		(property "LCSC" "C8678"
+			(at 157.48 62.865 90)
+			(effects
+				(font
+					(size 1.27 1.27)
+				)
+				(hide yes)
+			)
+		)
 		(pin "1"
 		)
@@
 			)
 		)
+		(property "LCSC" "C8678"
+			(at 157.48 104.775 90)
+			(effects
+				(font
+					(size 1.27 1.27)
+				)
+				(hide yes)
+			)
+		)
 		(pin "1"
 		)
@@
 			)
 		)
+		(property "LCSC" "C8678"
+			(at 157.48 90.17 90)
+			(effects
+				(font
+					(size 1.27 1.27)
+				)
+				(hide yes)
+			)
+		)
 		(pin "1"
 		)
@@
 			)
 		)
-		(property "LCSC_ext" "0"
-			(at 109.22 83.82 0)
-			(effects
-				(font
-					(size 1.27 1.27)
-				)
-				(hide yes)
-			)
-		)
 		(pin "1"
 		)
@@
 			)
 		)
+		(property "LCSC" "C8678"
+			(at 157.48 48.26 90)
+			(effects
+				(font
+					(size 1.27 1.27)
+				)
+				(hide yes)
+			)
+		)
 		(pin "1"
 		)
@@
 			(at 99.06 96.52 0)
 			(effects
-				(font
-					(size 1.27 1.27)
-				)
-				(hide yes)
-			)
-		)
-		(property "LCSC_ext" "0"
-			(at 99.06 96.52 0)
-			(effects

Commit message: bump modules
Connections:
- no-connect marks 0 -> 4
Changed lines of the file:
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@@
 		(color 0 0 0 0)
+	)
+	(no_connect
+		(at 128.905 109.855)
+	)
+	(no_connect
+		(at 128.27 67.945)
+	)
+	(no_connect
+		(at 129.54 95.25)
+	)
+	(no_connect
+		(at 127 53.34)
 	)
 	(wire
